Commit message: fix(urdf): mesh folder path

File: modules/g7_openarm_mujoco/src/g7_openarm_mujoco/model/urdf/g7_openarm.urdf (robot description, URDF)
Before this commit: robot g7_openarm, 31 links, 30 joints
Links:
- link AMR_FLW_link: geometry collision cylinder length=0.075 radius=0.052; visual mesh filename=../meshes/AMR_FLW_link.STL
- link AMR_FL_link: geometry visual mesh filename=../meshes/AMR_FL_link.STL
- link AMR_FRW_link: geometry collision cylinder length=0.075 radius=0.052; visual mesh filename=../meshes/AMR_FRW_link.STL
- link AMR_FR_link: geometry visual mesh filename=../meshes/AMR_FR_link.STL
- link AMR_RLW_link: geometry collision cylinder length=0.075 radius=0.052; visual mesh filename=../meshes/AMR_RLW_link.STL
- link AMR_RL_link: geometry visual mesh filename=../meshes/AMR_RL_link.STL
- link AMR_RRW_link: geometry collision cylinder length=0.075 radius=0.052; visual mesh filename=../meshes/AMR_RRW_link.STL
- link AMR_RR_link: geometry visual mesh filename=../meshes/AMR_RR_link.STL
- link AMR_base_link: geometry collision mesh filename=../meshes/AMR_base_link_collision.STL; visual mesh filename=../meshes/AMR_base_link.STL
- link L_link1: geometry collision mesh filename=../meshes/shoulder_L_link_collision.STL; visual mesh filename=../meshes/L_link1.STL
- link L_link2: geometry visual mesh filename=../meshes/L_link2.STL
- link L_link3: geometry collision mesh filename=../meshes/upper_arm_L_link_collision.STL; visual mesh filename=../meshes/L_link3.STL
- link L_link4: geometry collision mesh filename=../meshes/lower_arm_L_link_collision.STL; visual mesh filename=../meshes/L_link4.STL
- link L_link5: geometry collision mesh filename=../meshes/wrist1_L_link_collision.STL; visual mesh filename=../meshes/L_link5.STL
- link L_link6: geometry collision mesh filename=../meshes/L_link6_collision.STL; visual mesh filename=../meshes/L_link6.STL
- link L_link7: geometry collision mesh filename=../meshes/L_link7_collision.STL; visual mesh filename=../meshes/L_link7.STL
- link R_link1: geometry collision mesh filename=../meshes/shoulder_R_link_collision.STL; visual mesh filename=../meshes/R_link1.STL
- link R_link2: geometry visual mesh filename=../meshes/R_link2.STL
- link R_link3: geometry collision mesh filename=../meshes/upper_arm_L_link_collision.STL; visual mesh filename=../meshes/R_link3.STL
- link R_link4: geometry collision mesh filename=../meshes/lower_arm_L_link_collision.STL; visual mesh filename=../meshes/R_link4.STL
- link R_link5: geometry collision mesh filename=../meshes/wrist1_L_link_collision.STL; visual mesh filename=../meshes/R_link5.STL
- link R_link6: geometry collision mesh filename=../meshes/L_link6_collision.STL; visual mesh filename=../meshes/R_link6.STL
- link R_link7: geometry collision mesh filename=../meshes/R_link7_collision.STL; visual mesh filename=../meshes/R_link7.STL
- link chest_link: geometry collision mesh filename=../meshes/chest_link_collision.STL; visual mesh filename=../meshes/chest_link.STL
- link gripper_LL_link: geometry collision mesh filename=../meshes/gripper_LL_link_collision.STL; visual mesh filename=../meshes/gripper_LL_link.STL
- link gripper_LR_link: geometry collision mesh filename=../meshes/gripper_LR_link_collision.STL; visual mesh filename=../meshes/gripper_LR_link.STL
- link gripper_RL_link: geometry collision mesh filename=../meshes/gripper_RL_link_collision.STL; visual mesh filename=../meshes/gripper_RL_link.STL
- link gripper_RR_link: geometry collision mesh filename=../meshes/gripper_RR_link_collision.STL; visual mesh filename=../meshes/gripper_RR_link.STL
- link openarm_base_link: geometry collision mesh filename=../meshes/openarm_base_link_collision.STL; visual mesh filename=../meshes/openarm_base_link.STL

Commit message: chore(model): update MuJoCo and URDF robot models

File: modules/g7_openarm_mujoco/src/g7_openarm_mujoco/model/urdf/g7_openarm.urdf (robot description, URDF)
Before this commit: robot g7_openarm, 31 links, 30 joints
Links:
- removed link L_gripper_tcp_link
- removed link R_gripper_tcp_link
- added link L_tcp
- added link R_tcp
- link AMR_FLW_link: geometry collision cylinder length=0.075 radius=0.052; visual mesh filename=../meshes/AMR_FLW_link.stl
- link AMR_FL_link: geometry visual mesh filename=../meshes/AMR_FL_link.stl
- link AMR_FRW_link: geometry collision cylinder length=0.075 radius=0.052; visual mesh filename=../meshes/AMR_FRW_link.stl
- link AMR_FR_link: geometry visual mesh filename=../meshes/AMR_FR_link.stl
- link AMR_RLW_link: geometry collision cylinder length=0.075 radius=0.052; visual mesh filename=../meshes/AMR_RLW_link.stl
- link AMR_RL_link: geometry visual mesh filename=../meshes/AMR_RL_link.stl
- link AMR_RRW_link: geometry collision cylinder length=0.075 radius=0.052; visual mesh filename=../meshes/AMR_RRW_link.stl
- link AMR_RR_link: geometry visual mesh filename=../meshes/AMR_RR_link.stl
- link AMR_base_link: geometry collision mesh filename=../meshes/AMR_base_link_collision.stl; visual mesh filename=../meshes/AMR_base_link.stl
- link L_link1: geometry collision mesh filename=../meshes/shoulder_L_link_collision.stl; visual mesh filename=../meshes/L_link1.stl
- link L_link2: geometry visual mesh filename=../meshes/L_link2.stl
- link L_link3: geometry collision mesh filename=../meshes/upper_arm_L_link_collision.stl; visual mesh filename=../meshes/L_link3.stl
- link L_link4: geometry collision mesh filename=../meshes/lower_arm_L_link_collision.stl; visual mesh filename=../meshes/L_link4.stl
- link L_link5: geometry collision mesh filename=../meshes/wrist1_L_link_collision.stl; visual mesh filename=../meshes/L_link5.stl
- link L_link6: geometry collision mesh filename=../meshes/L_link6_collision.stl; visual mesh filename=../meshes/L_link6.stl
- link L_link7: mass 0.46500000 -> 0.63; geometry collision mesh filename=../meshes/gripper_L_link_collision.stl; visual mesh filename=../meshes/gripper_L_link.stl
- link R_link1: geometry collision mesh filename=../meshes/shoulder_R_link_collision.stl; visual mesh filename=../meshes/R_link1.stl
- link R_link2: geometry visual mesh filename=../meshes/R_link2.stl
- link R_link3: geometry collision mesh filename=../meshes/upper_arm_L_link_collision.stl; visual mesh filename=../meshes/R_link3.stl
- link R_link4: geometry collision mesh filename=../meshes/lower_arm_L_link_collision.stl; visual mesh filename=../meshes/R_link4.stl
- link R_link5: geometry collision mesh filename=../meshes/wrist1_L_link_collision.stl; visual mesh filename=../meshes/R_link5.stl
- link R_link6: geometry collision mesh filename=../meshes/L_link6_collision.stl; visual mesh filename=../meshes/R_link6.stl
- link R_link7: mass 0.46500000 -> 0.63; geometry collision mesh filename=../meshes/gripper_R_link_collision.stl; visual mesh filename=../meshes/gripper_R_link.stl
- link chest_link: mass 6.17600000 -> 2.28645698865; geometry collision mesh filename=../meshes/chest_link_collision.stl; visual mesh filename=../meshes/chest_link.stl
- link gripper_LL_link: mass 0.05000000 -> 0.12; geometry collision mesh filename=../meshes/gripper_LL_link_collision.stl; visual mesh filename=../meshes/gripper_LL_link.stl
- link gripper_LR_link: mass 0.05000000 -> 0.12; geometry collision mesh filename=../meshes/gripper_LR_link_collision.stl; visual mesh filename=../meshes/gripper_LR_link.stl
- link gripper_RL_link: mass 0.05000000 -> 0.12; geometry collision mesh filename=../meshes/gripper_RL_link_collision.stl; visual mesh filename=../meshes/gripper_RL_link.stl
- link gripper_RR_link: mass 0.05000000 -> 0.12; geometry collision mesh filename=../meshes/gripper_RR_link_collision.stl; visual mesh filename=../meshes/gripper_RR_link.stl
- link openarm_base_link: mass 10.00000000 -> 13.89; geometry collision mesh filename=../meshes/openarm_base_link_collision.stl; visual mesh filename=../meshes/openarm_base_link.stl
Joints:
- removed joint L_gripper_tcp_joint
- removed joint R_gripper_tcp_joint
- added joint L_tcp_joint: type fixed, parent L_link7, child L_tcp, origin xyz=-0.00102 -0.03226 -0.20576 rpy=3.141592653589793 0 -1.570796326794897
- added joint R_tcp_joint: type fixed, parent R_link7, child R_tcp, origin xyz=-0.00103 0.03132 -0.20576 rpy=3.141592653589793 0 1.570796326794897
- joint AMR_FLW_joint: limit effort=20 velocity=10 -> effort=15 velocity=10; type revolute -> continuous
- joint AMR_FRW_joint: limit effort=20 velocity=10 -> effort=15 velocity=10; type revolute -> continuous
- joint AMR_RLW_joint: limit effort=20 velocity=10 -> effort=15 velocity=10; type revolute -> continuous
- joint AMR_RRW_joint: limit effort=20 velocity=10 -> effort=15 velocity=10; type revolute -> continuous
- joint gripper_LL_joint: axis 0 1 0 -> -1 0 0; limit lower=0.0 upper=0.045 effort=20 velocity=0.1 -> lower=0 upper=0.045 effort=15 velocity=0.1; origin xyz=0 -0.01425 -0.119 rpy=0 0 0 -> xyz=-0.001886802417 0.012799907 -0.05450003114 rpy=-1.570784899 1.376982741e-06 1.570804785
- joint gripper_LR_joint: axis 0 -1 0 -> 1 0 0; limit lower=0.0 upper=0.045 effort=20 velocity=0.1 -> lower=0 upper=0.045 effort=15 velocity=0.1; origin xyz=0 -0.04925 -0.119 rpy=0 0 0 -> xyz=-0.002086032739 -0.07820009469 -0.05449990502 rpy=-1.570784899 1.376982741e-06 1.570804785
- joint gripper_RL_joint: axis 0 1 0 -> -1 0 0; limit lower=0.0 upper=0.045 effort=20 velocity=0.1 -> lower=0 upper=0.045 effort=15 velocity=0.1; origin xyz=0 0.04925 -0.119 rpy=0 0 0 -> xyz=-0.0002002716942 -0.00474640126 -0.05450008857 rpy=-1.570802202 7.72037562e-06 -1.570808101
- joint gripper_RR_joint: axis 0 -1 0 -> 1 0 0; limit lower=0.0 upper=0.045 effort=20 velocity=0.1 -> lower=0 upper=0.045 effort=15 velocity=0.1; origin xyz=0 0.01425 -0.119 rpy=0 0 0 -> xyz=-0.0001994122686 0.06824709873 -0.05450006127 rpy=-1.570802202 7.72037562e-06 -1.570808101

Commit message: Refactor code structure and remove redundant changes

File: modules/g7_openarm_mujoco/src/g7_openarm_mujoco/model/urdf/g7_openarm.urdf (robot description, URDF)
Before this commit: robot g7_openarm, 31 links, 30 joints
Links:
- removed link L_link8_L
- removed link L_link8_R
- removed link R_link8_L
- removed link R_link8_R
- added link gripper_LL_link, mass 0.12; collision mesh filename=../meshes/gripper_LL_link_collision.stl; visual mesh filename=../meshes/gripper_LL_link.stl
- added link gripper_LR_link, mass 0.12; collision mesh filename=../meshes/gripper_LR_link_collision.stl; visual mesh filename=../meshes/gripper_LR_link.stl
- added link gripper_RL_link, mass 0.12; collision mesh filename=../meshes/gripper_RL_link_collision.stl; visual mesh filename=../meshes/gripper_RL_link.stl
- added link gripper_RR_link, mass 0.12; collision mesh filename=../meshes/gripper_RR_link_collision.stl; visual mesh filename=../meshes/gripper_RR_link.stl
- added link head_base_link, mass 0.0288553383340636; collision mesh filename=../meshes/base_link.STL; visual mesh filename=../meshes/base_link.STL
- added link head_camera_link
- added link head_camera_optical_frame
- added link head_eye_link, mass 0.10791; collision mesh filename=../meshes/eye_Link.STL; visual mesh filename=../meshes/eye_Link.STL
- added link head_pitch_link, mass 0.180865339049976; collision mesh filename=../meshes/pitch_Link.STL; visual mesh filename=../meshes/pitch_Link.STL
- added link head_yaw_link, mass 0.21377; collision mesh filename=../meshes/yaw_Link.STL; visual mesh filename=../meshes/yaw_Link.STL
- link L_link7: geometry collision mesh filename=../meshes/gripper_L_link_collision.stl; visual mesh filename=../meshes/gripper_L_link.stl
- link R_link7: geometry collision mesh filename=../meshes/gripper_R_link_collision.stl; visual mesh filename=../meshes/gripper_R_link.stl
Joints:
- removed joint L_8_L_joint
- removed joint L_8_R_joint
- removed joint R_8_L_joint
- removed joint R_8_R_joint
- added joint gripper_LL_joint: type prismatic, parent L_link7, child gripper_LL_link, origin xyz=-0.001886802417 0.012799907 -0.05450003114 rpy=-1.570784899 1.376982741e-06 1.570804785, axis -1 0 0, limit lower=0 upper=0.045 effort=15 velocity=0.1
- added joint gripper_LR_joint: type prismatic, parent L_link7, child gripper_LR_link, origin xyz=-0.002086032739 -0.07820009469 -0.05449990502 rpy=-1.570784899 1.376982741e-06 1.570804785, axis 1 0 0, limit lower=0 upper=0.045 effort=15 velocity=0.1
- added joint gripper_RL_joint: type prismatic, parent R_link7, child gripper_RL_link, origin xyz=-0.0002002716942 -0.00474640126 -0.05450008857 rpy=-1.570802202 7.72037562e-06 -1.570808101, axis -1 0 0, limit lower=0 upper=0.045 effort=15 velocity=0.1
- added joint gripper_RR_joint: type prismatic, parent R_link7, child gripper_RR_link, origin xyz=-0.0001994122686 0.06824709873 -0.05450006127 rpy=-1.570802202 7.72037562e-06 -1.570808101, axis 1 0 0, limit lower=0 upper=0.045 effort=15 velocity=0.1
- added joint head_camera_mount_joint: type fixed, parent head_eye_link, child head_camera_link, origin xyz=0 0 0 rpy=0 0 0
- added joint head_camera_optical_joint: type fixed, parent head_camera_link, child head_camera_optical_frame, origin xyz=0 0 0 rpy=-1.57079632679 0 -1.57079632679
- added joint head_eye_joint: type fixed, parent head_pitch_link, child head_eye_link, origin xyz=0.079703 -0.023818 0.0031558 rpy=0 0 0, axis 0 0 0
- added joint head_mount_joint: type fixed, parent chest_link, child head_base_link, origin xyz=0 0 0.063 rpy=0 0 0
- added joint head_pitch_joint: type revolute, parent head_yaw_link, child head_pitch_link, origin xyz=0 0.02775 0.0385 rpy=0 0 0, axis 0 -1 0, limit lower=-0.7854 upper=0.7854 effort=5 velocity=2.0
- added joint head_yaw_joint: type revolute, parent head_base_link, child head_yaw_link, origin xyz=0 0 0.06 rpy=0 0 0, axis 0 0 1, limit lower=-1.5708 upper=1.5708 effort=5 velocity=2.0

Commit message: fix(mjcf): rename to correct filename

File: modules/g7_openarm_mujoco/src/g7_openarm_mujoco/model/urdf/g7_openarm.urdf (robot description, URDF)
Before this commit: robot g7_openarm, 37 links, 36 joints
Links:
- removed link gripper_LL_link
- removed link gripper_LR_link
- removed link gripper_RL_link
- removed link gripper_RR_link
- added link L_link8_L, mass 0.12; collision mesh filename=../meshes/L_link8_L_collision.stl; visual mesh filename=../meshes/L_link8_L.stl
- added link L_link8_R, mass 0.12; collision mesh filename=../meshes/L_link8_R_collision.stl; visual mesh filename=../meshes/L_link8_R.stl
- added link R_link8_L, mass 0.12; collision mesh filename=../meshes/R_link8_L_collision.stl; visual mesh filename=../meshes/R_link8_L.stl
- added link R_link8_R, mass 0.12; collision mesh filename=../meshes/R_link8_R_collision.stl; visual mesh filename=../meshes/R_link8_R.stl
- link L_link7: geometry collision mesh filename=../meshes/L_link7_collision.stl; visual mesh filename=../meshes/L_link7.stl
- link R_link7: geometry collision mesh filename=../meshes/R_link7_collision.stl; visual mesh filename=../meshes/R_link7.stl
Joints:
- removed joint gripper_LL_joint
- removed joint gripper_LR_joint
- removed joint gripper_RL_joint
- removed joint gripper_RR_joint
- added joint L_8_L_joint: type prismatic, parent L_link7, child L_link8_L, origin xyz=-0.001886802417 0.012799907 -0.05450003114 rpy=-1.570784899 1.376982741e-06 1.570804785, axis -1 0 0, limit lower=0 upper=0.045 effort=15 velocity=0.1
- added joint L_8_R_joint: type prismatic, parent L_link7, child L_link8_R, origin xyz=-0.002086032739 -0.07820009469 -0.05449990502 rpy=-1.570784899 1.376982741e-06 1.570804785, axis 1 0 0, limit lower=0 upper=0.045 effort=15 velocity=0.1
- added joint R_8_L_joint: type prismatic, parent R_link7, child R_link8_L, origin xyz=-0.0002002716942 -0.00474640126 -0.05450008857 rpy=-1.570802202 7.72037562e-06 -1.570808101, axis -1 0 0, limit lower=0 upper=0.045 effort=15 velocity=0.1
- added joint R_8_R_joint: type prismatic, parent R_link7, child R_link8_R, origin xyz=-0.0001994122686 0.06824709873 -0.05450006127 rpy=-1.570802202 7.72037562e-06 -1.570808101, axis 1 0 0, limit lower=0 upper=0.045 effort=15 velocity=0.1

Commit message: refactor: update joint dynamics parameters and improve visual material colors for left and right links

File: modules/g7_openarm_mujoco/src/g7_openarm_mujoco/model/urdf/g7_openarm.urdf (robot description, URDF)
Before this commit: robot g7_openarm, 37 links, 36 joints
Joints:
- joint L_7_joint: origin xyz=0 0.031749999999996 0 rpy=0 0 0 -> xyz=0 0.031749999999996 0 rpy=0 -0.2 0
- joint R_7_joint: origin xyz=0 -0.0317999999999935 0 rpy=0 0 0 -> xyz=0 -0.0317999999999935 0 rpy=0 -0.2 0

Commit message: refactor: mujoco, urdf model

File: modules/g7_openarm_mujoco/src/g7_openarm_mujoco/model/urdf/g7_openarm.urdf (robot description, URDF)
Before this commit: robot g7_openarm, 37 links, 36 joints
Joints:
- joint L_7_joint: origin xyz=0 0.031749999999996 0 rpy=0 -0.2 0 -> xyz=0 0.031749999999996 0 rpy=0 0 0
- joint R_7_joint: origin xyz=0 -0.0317999999999935 0 rpy=0 -0.2 0 -> xyz=0 -0.0317999999999935 0 rpy=0 0 0

Commit message: refactor: rename head link and joint and add rgb joint

File: modules/g7_openarm_mujoco/src/g7_openarm_mujoco/model/urdf/g7_openarm.urdf (robot description, URDF)
Before this commit: robot g7_openarm, 37 links, 36 joints
Links:
- removed link head_base_link
- removed link head_camera_link
- removed link head_camera_optical_frame
- removed link head_eye_link
- removed link head_pitch_link
- removed link head_yaw_link
- added link HEAD_base_link, mass 0.0288553383340636; collision mesh filename=../meshes/base_link.STL; visual mesh filename=../meshes/base_link.STL
- added link HEAD_camera_link
- added link HEAD_camera_optical_frame
- added link HEAD_color_link
- added link HEAD_color_optical_frame
- added link HEAD_eye_link, mass 0.10791; collision mesh filename=../meshes/eye_Link.STL; visual mesh filename=../meshes/eye_Link.STL
- added link HEAD_infra2_link
- added link HEAD_infra2_optical_frame
- added link HEAD_pitch_link, mass 0.180865339049976; collision mesh filename=../meshes/pitch_Link.STL; visual mesh filename=../meshes/pitch_Link.STL
- added link HEAD_yaw_link, mass 0.21377; collision mesh filename=../meshes/yaw_Link.STL; visual mesh filename=../meshes/yaw_Link.STL
Joints:
- removed joint head_camera_mount_joint
- removed joint head_camera_optical_joint
- removed joint head_eye_joint
- removed joint head_mount_joint
- removed joint head_pitch_joint
- removed joint head_yaw_joint
- added joint HEAD_camera_mount_joint: type fixed, parent HEAD_eye_link, child HEAD_camera_link, origin xyz=0.0009 0.0135 0 rpy=0 0 0
- added joint HEAD_camera_optical_joint: type fixed, parent HEAD_camera_link, child HEAD_camera_optical_frame, origin xyz=0 0 0 rpy=-1.57079632679 0 -1.57079632679
- added joint HEAD_color_mount_joint: type fixed, parent HEAD_camera_link, child HEAD_color_link, origin xyz=0 -0.015 0 rpy=0 0 0
- added joint HEAD_color_optical_joint: type fixed, parent HEAD_color_link, child HEAD_color_optical_frame, origin xyz=0 0 0 rpy=-1.57079632679 0 -1.57079632679
- added joint HEAD_eye_joint: type fixed, parent HEAD_pitch_link, child HEAD_eye_link, origin xyz=0.079703 -0.023818 0.0031558 rpy=0 0 0, axis 0 0 0
- added joint HEAD_infra2_mount_joint: type fixed, parent HEAD_camera_link, child HEAD_infra2_link, origin xyz=0 0.05 0 rpy=0 0 0
- added joint HEAD_infra2_optical_joint: type fixed, parent HEAD_infra2_link, child HEAD_infra2_optical_frame, origin xyz=0 0 0 rpy=-1.57079632679 0 -1.57079632679
- added joint HEAD_mount_joint: type fixed, parent chest_link, child HEAD_base_link, origin xyz=0 0 0.063 rpy=0 0 0
- added joint HEAD_pitch_joint: type revolute, parent HEAD_yaw_link, child HEAD_pitch_link, origin xyz=0 0.02775 0.0385 rpy=0 0 0, axis 0 -1 0, limit lower=-3.1415926535897931 upper=3.1415926535897931 effort=5 velocity=2.0
- added joint HEAD_yaw_joint: type revolute, parent HEAD_base_link, child HEAD_yaw_link, origin xyz=0 0 0.06 rpy=0 0 0, axis 0 0 1, limit lower=-1.5707963267948966 upper=1.5707963267948966 effort=5 velocity=2.0

File: modules/g7_openarm_mujoco/src/g7_openarm_mujoco/model/urdf/g7_openarm_pinnzoo.urdf (robot description, URDF)
Before this commit: robot g7_openarm, 37 links, 36 joints
Links:
- removed link head_base_link
- removed link head_camera_link
- removed link head_camera_optical_frame
- removed link head_eye_link
- removed link head_pitch_link
- removed link head_yaw_link
- added link HEAD_base_link, mass 0.0288553383340636; collision mesh filename=../meshes/base_link.STL; visual mesh filename=../meshes/base_link.STL
- added link HEAD_camera_link
- added link HEAD_camera_optical_frame
- added link HEAD_color_link
- added link HEAD_color_optical_frame
- added link HEAD_eye_link, mass 0.10791; collision mesh filename=../meshes/eye_Link.STL; visual mesh filename=../meshes/eye_Link.STL
- added link HEAD_infra2_link
- added link HEAD_infra2_optical_frame
- added link HEAD_pitch_link, mass 0.180865339049976; collision mesh filename=../meshes/pitch_Link.STL; visual mesh filename=../meshes/pitch_Link.STL
- added link HEAD_yaw_link, mass 0.21377; collision mesh filename=../meshes/yaw_Link.STL; visual mesh filename=../meshes/yaw_Link.STL
Joints:
- removed joint head_camera_mount_joint
- removed joint head_camera_optical_joint
- removed joint head_eye_joint
- removed joint head_mount_joint
- removed joint head_pitch_joint
- removed joint head_yaw_joint
- added joint HEAD_camera_mount_joint: type fixed, parent HEAD_eye_link, child HEAD_camera_link, origin xyz=0.0009 0.0135 0 rpy=0 0 0
- added joint HEAD_camera_optical_joint: type fixed, parent HEAD_camera_link, child HEAD_camera_optical_frame, origin xyz=0 0 0 rpy=-1.57079632679 0 -1.57079632679
- added joint HEAD_color_mount_joint: type fixed, parent HEAD_camera_link, child HEAD_color_link, origin xyz=0 -0.015 0 rpy=0 0 0
- added joint HEAD_color_optical_joint: type fixed, parent HEAD_color_link, child HEAD_color_optical_frame, origin xyz=0 0 0 rpy=-1.57079632679 0 -1.57079632679
- added joint HEAD_eye_joint: type fixed, parent HEAD_pitch_link, child HEAD_eye_link, origin xyz=0.079703 -0.023818 0.0031558 rpy=0 0 0, axis 0 0 0
- added joint HEAD_infra2_mount_joint: type fixed, parent HEAD_camera_link, child HEAD_infra2_link, origin xyz=0 0.05 0 rpy=0 0 0
- added joint HEAD_infra2_optical_joint: type fixed, parent HEAD_infra2_link, child HEAD_infra2_optical_frame, origin xyz=0 0 0 rpy=-1.57079632679 0 -1.57079632679
- added joint HEAD_mount_joint: type fixed, parent chest_link, child HEAD_base_link, origin xyz=0 0 0.063 rpy=0 0 0
- added joint HEAD_pitch_joint: type revolute, parent HEAD_yaw_link, child HEAD_pitch_link, origin xyz=0 0.02775 0.0385 rpy=0 0 0, axis 0 -1 0, limit lower=-3.1415926535897931 upper=3.1415926535897931 effort=5 velocity=2.0
- added joint HEAD_yaw_joint: type revolute, parent HEAD_base_link, child HEAD_yaw_link, origin xyz=0 0 0.06 rpy=0 0 0, axis 0 0 1, limit lower=-1.5707963267948966 upper=1.5707963267948966 effort=5 velocity=2.0
